File: Krakatau Board v1.3.brd (EAGLE design)
At the start: 81 x 120 mm, 134 parts, among them J1 MMCX-P-P-X-ST-TH1, J12 SAMTEC-CLP-110-02-X-D, J2 MMCX-P-P-X-ST-TH1, J8 61300511121, SW1 TL3342F160QG, T1 SUM110P06-07L-E3, U1 STM32F413VHT6, U10 TESEO-LIV3F, U11 BGA725L6E6327FTSA1, U12 DS3231S, U13 24LC01B, U14 LTC4151IMS, U15 MMBT2907ALT1GSOT-23-3D, U16 IIS328DQ, U2 LM3671MF-3.3, U3 LMR33630ADDAR, U4 REF2933AIDBZR, U5 BT832X, U6 MAX232E, U7 MAX232E, U8 FT234XD-R, U9 MAX5490, Y1 ECS-250-20-33-CKM-TR, Y2 ECS-.327-12.5-34B-TR, Y3 U.FL, Y4 U.FL, Y5 U.FL

Commit message: finalisasi
Parts:
- added SUPPLY3, SUPPLY4, SUPPLY5, SUPPLY6, SUPPLY7: 2PT_GND_TIE, SparkFun-PowerSymbols:2PT_GND_TIE
- moved C60 38.1 mm to (16.3, 45.5), turned to 0 degrees
- moved R14 38.1 mm to (15.4, 51.4), turned to 90 degrees
- moved U13 37.2 mm to (16.4, 48.3), turned to 180 degrees
- moved R13 35.4 mm to (17.3, 51.4), turned to 90 degrees
- moved C42 23.5 mm to (8.44, 22.8)
- moved C43 22.2 mm to (12.4, 22.7), turned to 90 degrees
- moved C40 21.2 mm to (6.52, 22.8), turned to 90 degrees
- moved C41 20.0 mm to (10.4, 22.7), turned to 90 degrees
- moved C35 19.3 mm to (23.6, 22.8), turned to 90 degrees
- moved C34 18.3 mm to (19.7, 22.9), turned to 90 degrees
- moved C37 17.3 mm to (25.5, 22.8), turned to 90 degrees
- moved C36 16.5 mm to (21.6, 22.9)
- moved U7 14.7 mm to (10.9, 15.2)
- moved C9 13.8 mm to (39.0, 40.7), turned to 0 degrees
- moved C39 13.7 mm to (7.14, 8.00), turned to 180 degrees
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Connections:
- net N$43 renamed DP
- net N$44 renamed DM
- removed net CS_ACC: U16.12
- removed net INT1_ACC: U16.7
- removed net INT2_ACC: U16.3
- removed net N$105: U10.17
- removed net N$106: U10.16
- removed net N$109: R12.1, U12.3
- removed net N$110: U10.9
- removed net N$111: R10.1, U12.15
- removed net N$112: R11.1, U12.16
- removed net N$113: R13.1, U13.SDA
- removed net N$114: R14.1, U13.SCL
- removed net N$116: R15.1, U14.7
- removed net N$117: R16.1, U14.6
- removed net N$122: R21.1
- removed net N$20: U1.97
- removed net N$25: U1.92
- removed net N$26: U1.91
- removed net N$27: U1.90
- removed net N$28: U1.89
- removed net N$29: U1.88
- removed net N$3: C3.1, SW1.3, SW1.4
- removed net N$30: U1.87
- removed net N$31: U1.86
- removed net N$32: U1.85
- removed net N$33: U1.84
- removed net N$34: U1.83
- removed net N$35: U1.82
- removed net N$36: U1.81
- removed net N$37: U1.80
- removed net N$38: U1.79
- removed net N$39: U1.78
- removed net N$4: C5.1, Y1.1
- removed net N$40: U1.77
- removed net N$45: U1.69
- removed net N$46: U1.68
- removed net N$47: U1.65
- removed net N$48: U1.64
- removed net N$49: U1.63
- removed net N$5: C4.1, Y1.3
- removed net N$50: U1.62
- removed net N$51: U1.61
- removed net N$52: U1.60
- removed net N$53: U1.59
- removed net N$54: U1.58
- removed net N$55: U1.57
- removed net N$56: U1.56
- removed net N$57: U1.55
- removed net N$58: U1.54
- removed net N$59: U1.53
- removed net N$60: U1.52
- removed net N$61: U1.51
- removed net N$64: U9.3
- removed net N$74: U7.14
- removed net N$75: U7.7
- removed net N$76: U7.13
- removed net N$77: U7.8
- removed net N$78: U7.11
- removed net N$79: U7.10
- removed net N$8: C7.1, Y2.1
- removed net N$80: U7.12
- removed net N$81: U7.9
- removed net N$82: U6.14
- removed net N$83: U6.7
- removed net N$84: U6.13
- removed net N$85: U6.8
- removed net N$86: U6.11
- removed net N$87: U6.10
- removed net N$88: U6.12
- removed net N$89: U6.9
- removed net N$9: C6.1, Y2.2
- removed net N$93: C53.2, U10.2
- removed net N$95: C52.2, U10.3
- removed net N$96: U8.7
- removed net N$97: U8.10
- removed net N$98: C54.2, U10.4
- removed net N$99: U10.5
- removed net SDI_ACC: U16.16
- removed net SDO_ACC: U16.15
- removed net SPC_ACC: U16.11
- new net ACC_INT1: U1.33, U16.7
- new net ACC_INT2: U1.34, U16.3
- new net ACC_MISO: U1.31, U16.15
- new net ACC_MOSI: U1.32, U16.16
- new net ACC_NSS: U1.29, U16.12
- new net ACC_SCK: U1.30, U16.11
- new net BATTSENSE: U1.16, U9.3
- new net CD: J10.9, U1.77
- new net EEPROM_SCL: R14.1, U1.92, U13.SCL
- new net EEPROM_SDA: R13.1, U1.93, U13.SDA
- new net GNDA: J1.2, J1.3, J1.4, J1.5, J2.2, J2.3, J2.4, J2.5, SUPPLY4.P$1, SUPPLY7.P$1, Y4.1, Y4.3, Y5.1, Y5.3
- new net GPS_PPS: C54.2, U1.40, U10.4
- new net GPS_RESET: U1.41, U10.9
- new net GPS_RX: C53.2, U1.38, U10.2
- new net GPS_TX: C52.2, U1.39, U10.3
- new net GPS_WAKEUP: U1.42, U10.5
- new net LEAKAGE: R21.1, U1.3
- new net LED: J13.2, U1.37
- new net OSC32_IN: C7.1, U1.8, Y2.1
- new net OSC32_OUT: C6.1, U1.9, Y2.2
- new net OSC_IN: C5.1, U1.12, Y1.1
- new net OSC_OUT: C4.1, U1.13, Y1.3
- new net POWER_SCL: R16.1, U1.67, U14.6
- new net POWER_SDA: R15.1, U1.90, U14.7
- new net RS232_1_RX: U1.97, U6.12
- new net RS232_1_TX: U1.98, U6.11
- new net RS232_2_RX: U1.26, U7.12
- new net RS232_2_TX: U1.25, U7.11
- new net RS232_3_RX: U1.24, U6.9
- new net RS232_3_TX: U1.23, U6.10
- new net RTC_INT1: R12.1, U1.69, U12.3
- new net RTC_SCL: R11.1, U1.47, U12.16
- new net RTC_SDA: R10.1, U1.89, U12.15
- new net SDIO_CK: J10.5, U1.80
- new net SDIO_CMD: J10.3, U1.83
- new net SDIO_D0: J10.7, U1.65
- new net SDIO_D1: J10.8, U1.66
- new net SDIO_D2: J10.1, U1.78
- new net SDIO_D3: J10.2, U1.79
- new net TTL_RX: J14.3, U1.1
- new net TTL_TX: J14.2, U1.2
- new net USB_RX: U1.51, U8.7
- new net USB_TX: U1.52, U8.10
- net +3V3: now also J10.4, U1.6
- net 0V: now also SUPPLY3.P$2, U14.4, U14.5, U14.9; no longer C25.2, C26.2, C27.2, C28.1, C29.1, C30.1, C32.2, C33.2, D1.2, J11.1, J3.1, R17.2, R4.1, U2.2, U3.1, U3.9, U4.3, U9.2
- net AGND: now also FL1.2, FL1.3, FL1.5, SUPPLY5.P$2, SUPPLY6.P$2, U10.1; no longer J1.2, J1.3, J1.4, J1.5, J2.2, J2.3, J2.4, J2.5, Y4.1, Y4.3, Y5.1, Y5.3
- net BT_CON: now also U1.62
- net BT_RX: now also U1.64
- net BT_TX: now also U1.63
- net CLK: now also J8.2
- net DF_CTS: now also U1.58
- net DF_DCD: now also U1.46
- net DF_DSR: now also U1.54
- net DF_DTR: now also U1.57
- net DF_RI: now also U1.53
- net DF_RTS: now also U1.59
- net DF_S_RX: now also U1.56
- net DF_S_TX: now also U1.55
- net DIO: now also J8.1
- net GND: now also C25.2, C26.2, C27.2, C28.1, C29.1, C30.1, C32.2, C33.2, D1.2, J10.10, J10.11, J10.12, J10.13, J10.6, J11.1, J13.1, J14.1, J3.1, J4.1, J6.1, J7.1, J8.4, J9.1, R17.2, R4.1, SUPPLY3.P$1, SUPPLY4.P$2, SUPPLY5.P$1, SUPPLY6.P$1, SUPPLY7.P$2, U2.2, U3.1, U3.9, U4.3, U9.2; no longer FL1.2, FL1.3, FL1.5, U10.1, U14.4, U14.5, U14.9
- net N$10: now also J6.3, U7.13; no longer U1.66
- net N$19: now also J4.2, U6.14; no longer U1.98
- net N$21: now also J4.3, U6.13; no longer U1.96
- net N$22: now also J7.2, U6.7; no longer U1.95
- net N$24: now also J7.3, U6.8; no longer U1.93
- net N$6: now also J6.2, U7.14; no longer U1.67
- net N$73: now also J9.3
- net N$90: now also J9.2
- net N$91: now also J9.4
- net NETWORKINT: now also U1.61
- net ON/OFF: now also U1.60
- net RST: now also C3.1, J8.3, SW1.3, SW1.4
- net VBAT: now also U10.6; no longer U1.6
Routing:
- net +3V3: track 56.9 -> 365.8 mm, vias 6 -> 12
- net +5V: track 21.1 -> 211.7 mm, vias 0 -> 2
- net POWER_SCL: track 0.00 -> 176.8 mm, vias 0 -> 4
- net POWER_SDA: track 0.00 -> 160.9 mm, vias 0 -> 4
- net SDIO_D0: track 0.00 -> 149.7 mm, vias 0 -> 1
- net SDIO_D1: track 0.00 -> 146.4 mm, vias 0 -> 1
- net TTL_TX: track 0.00 -> 135.7 mm, vias 0 -> 3
- net TTL_RX: track 0.00 -> 133.0 mm, vias 0 -> 3
- net VBAT: track 0.00 -> 128.6 mm, vias 0 -> 2
- net CD: track 0.00 -> 122.3 mm, vias 0 -> 1
- net SDIO_D2: track 0.00 -> 120.2 mm, vias 0 -> 1
- net SDIO_D3: track 0.00 -> 116.7 mm, vias 0 -> 1
- net SDIO_CK: track 0.00 -> 114.1 mm, vias 0 -> 1
- net SDIO_CMD: track 0.00 -> 108.9 mm, vias 0 -> 1
- net RS232_2_RX: track 0.00 -> 77.0 mm, vias 0 -> 3
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- added copper zone on layer 16, net AGND
- added copper zone on layer 1, net GNDA
- added copper zone on layer 16, net GNDA
Other:
- board text added: "Krakatau Board v1.3"
- board text removed: "Krakatau Board v1.4"

Commit message: vias 0.25 min pcbway for 2mm
Parts:
- removed SUPPLY3: 2PT_GND_TIE, SparkFun-PowerSymbols:2PT_GND_TIE
- added C63, C64: 22uF, LMK212BBJ226MD-T:CAPC2113X95N
- added J15: 61300311121, Headers:61300311121
- R4: value 24.9 -> 24.9K
- moved C29 1.70 mm to (68.5, 37.6)
- moved C30 1.60 mm to (75.1, 37.6)
Connections:
- removed net 0V: SUPPLY3.P$2, U14.4, U14.5, U14.9
- net BT_CLK: now also J15.2
- net BT_DIO: now also J15.1
- net BT_RESET: now also J15.3
- net GND: now also C63.1, C64.1, U14.4, U14.5, U14.9; no longer SUPPLY3.P$1
- net N$12: now also C63.2, C64.2
Routing:
- net BT_RESET: track 0.00 -> 32.2 mm, vias 0 -> 1
- net BT_CLK: track 0.00 -> 30.8 mm, vias 0 -> 1
- net BT_DIO: track 0.00 -> 29.2 mm, vias 0 -> 1
- net 0V: track 16.8 -> 0.00 mm, vias 2 -> 0
- net VBAT: track 128.6 -> 139.2 mm
- net GND: track 5.94 -> 16.0 mm, vias 65 -> 165
- net N$12: track 15.2 -> 18.1 mm
- net USB_RX: track 22.2 -> 22.9 mm
- removed copper zone on layer 1, net 0V
Other:
- board text added: "BT Firm"
- board text added: "BT-POWER"
- board text added: "CLK"
- board text added: "DEBUGGER"
- board text added: "DIO"
- board text added: "GPS POWER"
- board text added: "LED"
- board text added: "RST"
- board text added: "RX"
- board text added: "TTL"
- board text added: "TX"
